Commit message: TF tree updates

File: pumpkin_bot_description/src/description/pumpkin_bot_description.urdf (robot description, URDF)
Before this commit: robot pumpkin_bot, 5 links, 4 joints
Joints:
- removed joint base_joint
- added joint base_footprint_joint: type fixed, parent base_footprint, child base_link, origin xyz=0.0 0.0 0.09 rpy=0 0 0

Commit message: More Nav stuff

File: pumpkin_bot_description/src/description/pumpkin_bot_description.urdf (robot description, URDF)
Before this commit: robot pumpkin_bot, 5 links, 4 joints
Joints:
- joint imu_joint: origin xyz=-0.14 0 0.23 rpy=${pi} 0 ${pi/2} -> xyz=-0.14 0 0.23 rpy=0 0 0
